Commit message: Nav2/SLAM working!
Gazebo can fire up with 1 to 5 rovers that build dynamically a map

File: leo_common-ros2/leo_description/urdf/macros.xacro (robot description, xacro)
@@ -165,5 +165,16 @@
       </link>
     </xacro:if>
-    <!-- REALSENSE CAMERA LINK -->
+    <!-- ===== 2D LIDAR ===== -->
+    <link name="${link_prefix}lidar_link">
+      <visual>
+        <geometry>
+          <cylinder radius="0.04" length="0.03"/>
+        </geometry>
+        <material name="DarkGrey">
+          <color rgba="0.3 0.3 0.3 1"/>
+        </material>
+      </visual>
+    </link>
+    <!-- REALSENSE CAMERA LINK (active alongside LiDAR) -->
     <link name="${link_prefix}realsense_link">
       <visual>
@@ -263,4 +274,11 @@
       </joint>
     </xacro:if>
+    <!-- LiDAR mounted on top of base_link (360° view) -->
+    <joint name="${joint_prefix}lidar_joint" type="fixed">
+      <parent link="${link_prefix}base_link"/>
+      <child link="${link_prefix}lidar_link"/>
+      <origin xyz="0 0 0.1" rpy="0 0 0"/>
+    </joint>
+    <!-- REALSENSE JOINT (active alongside LiDAR) -->
     <joint name="${joint_prefix}realsense_joint" type="fixed">
       <parent link="${link_prefix}base_link"/>
@@ -427,4 +445,29 @@
       </collision>
     </gazebo>
+    <!-- ===== 2D LIDAR SENSOR (360°, replaces RealSense depth camera) ===== -->
+    <gazebo reference="${link_prefix}lidar_link">
+      <sensor name="lidar" type="gpu_lidar">
+        <always_on>1</always_on>
+        <update_rate>10</update_rate>
+        <lidar>
+          <scan>
+            <horizontal>
+              <samples>360</samples>
+              <resolution>1</resolution>
+              <min_angle>-3.14159</min_angle>
+              <max_angle>3.14159</max_angle>
+            </horizontal>
+          </scan>
+          <range>
+            <min>0.1</min>
+            <max>10.0</max>
+            <resolution>0.01</resolution>
+          </range>
+        </lidar>
+        <topic>${link_prefix}lidar/scan</topic>
+        <frame_id>lidar_link</frame_id>
+      </sensor>
+    </gazebo>
+    <!-- REALSENSE CAMERA SENSOR (active alongside LiDAR) -->
     <gazebo reference="${link_prefix}realsense_link">
       <sensor name="depth_camera" type="rgbd_camera">
@@ -435,10 +478,7 @@
           <lens>
             <intrinsics>
-              <!-- fx = fy = width / ( 2 * tan (hfov / 2 ) ) -->
               <fx>554.25469</fx>
               <fy>554.25469</fy>
-              <!-- cx = ( width + 1 ) / 2 -->
               <cx>320.5</cx>
-              <!-- cy = ( height + 1 ) / 2 -->
               <cy>240.5</cy>
               <s>0</s>
